File: kicad/MoonPhase.kicad_pcb (KiCad board)
At the start: 2 copper layers, 72.4 x 59.7 mm, 13 parts, among them J1 Conn_IL, J2 Conn_PV, J3 Conn_LS, U1 ULN2003A, U2 ULN2003A, U3 RaspberryPi_Pico_W

Commit message: PCB Rev B
Parts:
- added C1: 22uF 16v, Capacitor_THT:CP_Radial_D4.0mm_P2.00mm, F.Cu at (167.6, 108.0)
- added C2: 22uF 16v, Capacitor_THT:CP_Radial_D4.0mm_P2.00mm, F.Cu at (167.6, 112.5)
- moved G*** 22.9 mm to (167.6, 82.5)
- moved R1 3.45 mm to (167.6, 74.0)
- moved R2 2.81 mm to (167.6, 91.7)
- moved J3 2.46 mm to (177.1, 92.7)
Connections:
- U1 pad 10: unconnected-(U1-O7-Pad10) -> IL_OUT_1
- U1 pad 11: unconnected-(U1-O6-Pad11) -> IL_OUT_1
- U1 pad 6: unconnected-(U1-I6-Pad6) -> IL_IN_1
- U1 pad 7: unconnected-(U1-I7-Pad7) -> IL_IN_1
- U2 pad 12: IL_OUT_1 -> IL_OUT_2
- U2 pad 5: IL_IN_1 -> IL_IN_2
Routing:
- net IL_OUT_1: track 21.2 -> 43.6 mm
- net IL_IN_1: track 29.7 -> 51.0 mm
- net +5V: track 132.7 -> 146.1 mm
- net Net-(D1-K): track 5.77 -> 2.32 mm
- net Net-(D2-K): track 5.68 -> 2.87 mm
- net IL_IN_2: track 30.9 -> 33.4 mm
- net IL_OUT_2: track 21.2 -> 23.2 mm
- net LED_IN: track 50.4 -> 51.9 mm
- net LS_OUT_1: track 21.8 -> 20.5 mm
- net LS_OUT_4: track 19.9 -> 18.9 mm
- net LS_OUT_2: track 19.9 -> 18.8 mm
- net LS_OUT_3: track 19.9 -> 18.9 mm
- net PV_OUT_4: track 21.2 -> 20.4 mm
Other:
- board text added: "Moon Phase Display Rev B"
- board text removed: "Moon Phase Display Rev A"

Commit message: PCB Rev C Update
Parts:
- added Q1: Q_Photo_NPN, Connector_PinHeader_2.54mm:PinHeader_1x02_P2.54mm_Vertical, F.Cu at (147.0, 115.6)
- added R4: 10k, Resistor_SMD:R_0805_2012Metric, F.Cu at (147.3, 86.7)
Connections:
- U3 pad 31: unconnected-(U3-GPIO26_ADC0-Pad31)_1 -> Net-(Q1-C)
- U3 pad 36: unconnected-(U3-3V3-Pad36)_1 -> +3V3
Routing:
- net Net-(Q1-C): track 0.00 -> 35.5 mm
- net +3V3: track 0.00 -> 18.5 mm, vias 0 -> 1
- net GND: track 47.6 -> 52.0 mm
- net LED_IN: vias 0 -> 1
Other:
- board text added: "Moon Phase Display Rev C"
- board text removed: "Moon Phase Display Rev B"
