File: kicad/MoonPhase.kicad_sch (KiCad schematic)
At the start: 12 parts, among them J1 Conn_IL, J2 Conn_PV, J3 Conn_LS, U1 ULN2003A, U2 ULN2003A, U3 RaspberryPi_Pico_W

Commit message: PCB Rev B
Parts:
- added C1, C2: 22uF 16v, Capacitor_THT:CP_Radial_D4.0mm_P2.00mm, symbol Device:C_Polarized
Connections:
- net +5V: now also C1.1, C2.1
- net IL_IN_1: now also U1.6 (I6), U1.7 (I7); no longer U2.5 (I5)
- net IL_IN_2: now also U2.5 (I5)
- net IL_OUT_1: now also U1.10 (O7), U1.11 (O6), C1.2; no longer U2.12 (O5)
- net IL_OUT_2: now also U2.12 (O5), C2.2
- no-connect marks 27 -> 23

Commit message: PCB Rev C Update
Parts:
- added Q1: Q_Photo_NPN, Connector_PinHeader_2.54mm:PinHeader_1x02_P2.54mm_Vertical, symbol Device:Q_Photo_NPN
- added R4: 10k, Resistor_SMD:R_0805_2012Metric, symbol Device:R
Connections:
- net GND: now also Q1.2 (E)
- net at U3.31 (GPIO26_ADC0): now also Q1.1 (C), R4.2
- net +3V3: now reaches U3.36 (3V3)
- net +3V3: now also R4.1
- no-connect marks 23 -> 21
Other:
- moved on the sheet: U3
